File: Schematic/OPL3_VGM_Player/OPL3_VGM_Player.sch (KiCad schematic (older format))
At the start: 20 parts, among them J1 USB_OTG, U1 LD1117S33TR_SOT223, U2 STM32F103C8Tx, U3 CH340E

Commit message: Saving work on schematic. IO Pin Changes
Parts:
- added C12, C20: 100nF, symbol device:C_Small
- added C13, C19: 10uF, symbol device:CP_Small
- added C14, C15: C_Small, symbol device:C_Small
- added C16: 68pF, symbol device:C_Small
- added C17, C18: 2.7nF, symbol device:C_Small
- added J3: Micro_SD_Card, symbol conn:Micro_SD_Card
- added J4: Conn_01x04, symbol conn:Conn_01x04
- added L2: 33uH, symbol device:L_Small
- added R3: 1K, symbol device:R_Small
- added R4, R5: 10K, symbol device:R_Small
- added R6: 33, symbol device:R_Small
- added SW1: SW_Push_Dual, symbol switches:SW_Push_Dual
- added U4: YMF262-M, symbol OPL3:YMF262-M
- added U5: YAC512-M, symbol OPL3:YAC512-M
- added U6: TL074, symbol linear:TL074
- gave numbers to parts that had none: 9
Connections:
- net +3V3: now also C12.1, J3.4 (VDD), J4.1 (Pin_1), R4.1
- net +5V: now also C14.2, L2.2, R5.2, U4.1 (VDD)
- net GND: now also C12.2, C13.2, C14.1, C15.1, C16.1, C17.1, C18.1, C19.2, C20.1, J3.6 (VSS), J4.4 (Pin_4), R3.2, U4.12 (VSS), U5.2 (VSS), U6.11 (V-)
- net RX: now also U2.30 (TIM1_CH2/USART1_TX/PA9)
- net TX: now also U2.31 (TIM1_CH3/USART1_RX/PA10)
- net YM_CLK: now reaches U2.11 (ADC1_IN1/ADC2_IN1/TIM2_CH2/USART2_RTS/PA1)
- net YM_CLK: now also U4.24 (ØM)
- net SD_CS: now reaches U2.14 (ADC1_IN4/ADC2_IN4/SPI1_NSS/USART2_CK/PA4)
- net SD_CS: now also J3.2 (DAT3/CD)
- net SD_CLK: now reaches U2.15 (ADC1_IN5/ADC2_IN5/SPI1_SCK/PA5)
- net SD_CLK: now also J3.5 (CLK)
- net SD_MISO: now reaches U2.16 (ADC1_IN6/ADC2_IN6/SPI1_MISO/TIM1_BKIN/TIM3_CH1/PA6)
- net SD_MISO: now also J3.7 (DAT0)
- net SD_MOSI: now reaches U2.17 (ADC1_IN7/ADC2_IN7/SPI1_MOSI/TIM1_CH1N/TIM3_CH2/PA7)
- net SD_MOSI: now also J3.3 (CMD)
- net YM_A0: now reaches U2.2 (PC13/RTC_OUT/RTC_TAMPER)
- net YM_A0: now also U4.4 (A0)
- net D2: now reaches U2.21 (PB10/I2C2_SCL/TIM2_CH3/USART3_TX)
- net D2: now also U4.13 (D2)
- net D3: now reaches U2.22 (PB11/ADC1_EXTI11/ADC2_EXTI11/I2C2_SDA/TIM2_CH4/USART3_RX)
- net D3: now also U4.14 (D3)
- net D4: now reaches U2.25 (PB12/I2C2_SMBA/SPI2_NSS/TIM1_BKIN/USART3_CK)
- net D4: now also U4.15 (D4)
- net D5: now reaches U2.26 (PB13/SPI2_SCK/TIM1_CH1N/USART3_CTS)
- net D5: now also U4.16 (D5)
- net D6: now reaches U2.27 (PB14/SPI2_MISO/TIM1_CH2N/USART3_RTS)
- net D6: now also U4.17 (D6)
- net D7: now reaches U2.28 (PB15/ADC1_EXTI15/ADC2_EXTI15/SPI2_MOSI/TIM1_CH3N)
- net D7: now also U4.18 (D7)
- net YM_CS: now reaches U2.29 (RCC_MCO/TIM1_CH1/USART1_CK/PA8)
- net YM_CS: now also U4.8 (CS)
- net YM_A1: now reaches U2.3 (PC14/RCC_OSC32_IN)
- net YM_A1: now also U4.5 (A1)
- net SWDIO: now reaches U2.34 (SYS_JTMS-SWDIO/PA13)
- net SWDIO: now also J4.2 (Pin_2)
- net SWCLK: now reaches U2.37 (SYS_JTCK-SWCLK/PA14)
- net SWCLK: now also J4.3 (Pin_3)
- net YM_IC: now reaches U2.38 (ADC1_EXTI15/ADC2_EXTI15/SPI1_NSS/SYS_JTDI/TIM2_CH1/TIM2_ETR/PA15)
- net YM_IC: now also U4.3 (IC)
- net YM_WR: now reaches U2.41 (PB5/I2C1_SMBA/SPI1_MOSI/TIM3_CH2)
- net YM_WR: now also U4.6 (WR)
- net D0: now reaches U2.45 (PB8/CAN_RX/I2C1_SCL/TIM4_CH3)
- net D0: now also U4.10 (D0)
- net D1: now reaches U2.46 (PB9/CAN_TX/I2C1_SDA/TIM4_CH4)
- net D1: now also U4.11 (D1)
- net at U2.7 (NRST): now also R4.2, SW1.4
- new net: R5.1, U4.7 (RD)
- new net: R3.1, SW1.1
- new net: U4.19 (SMPBD), U5.8 (SMP1)
- new net: U4.20 (SMPAC), U5.7 (SMP2)
- new net: U4.21 (DOAB), U5.4 (DIN)
- new net: U4.23 (ØSY), U5.5 (CLK)
- new net: C17.2, U5.10 (CH1), U6.12 (+)
- new net: C18.2, U5.11 (CH2), U6.10 (+)
- new net: R6.2, U5.12 (SWIN)
- new net: C16.2, U5.13 (AOUT), U6.5 (+)
- new net: U5.14 (MP), U6.1, U6.2 (-)
- new net: C19.1, U5.16 (CV), U6.3 (+)
- new net: R6.1, U6.6 (-), U6.7
- new net +5VA: C13.1, C15.2, C20.2, L2.1, U5.1 (VDD), U5.3 (VDD), U5.6 (FSEL), U5.9 (TST1), U6.4 (V+)
- new net CH1_OUT: U6.13 (-), U6.14
- new net CH2_OUT: U6.8, U6.9 (-)
- no-connect marks 5 -> 14

Commit message: Schematic plotted
Parts:
- added C21: 10uF, symbol device:C_Small
- added C22, C23: 10uF, symbol device:CP_Small
- added DS1: 128x32_I2C_OLED, symbol oled:128x32_I2C_OLED
- added J5: Audio-Jack-3, symbol conn:Audio-Jack-3
- added L3: 10uH, symbol device:L_Small
- added R7: 4.7, symbol device:R_Small
- added R8, R9: 4.7K, symbol device:R_Small
- added RV1: R_POT_Dual, symbol device:R_POT_Dual
- added SW2, SW3, SW4, SW5: SW_Push_Dual, symbol switches:SW_Push_Dual
Connections:
- net +3V3: now also R7.2, R8.2, R9.2
- net CH1_OUT: now also C22.1
- net CH2_OUT: now also C23.1
- net GND: now also C21.2, DS1.4 (GND), J5.3, RV1.3, RV1.6, SW2.3, SW3.3, SW4.3, SW5.3
- net PREV: now reaches U2.18 (PB0/ADC1_IN8/ADC2_IN8/TIM1_CH2N/TIM3_CH3)
- net PREV: now also SW2.1
- net RAND: now reaches U2.19 (PB1/ADC1_IN9/ADC2_IN9/TIM1_CH3N/TIM3_CH4)
- net RAND: now also SW3.1
- net NEXT: now reaches U2.39 (PB3/SPI1_SCK/SYS_JTDO-TRACESWO/TIM2_CH2)
- net NEXT: now also SW4.1
- net OPTION: now reaches U2.40 (PB4/SPI1_MISO/SYS_NJTRST/TIM3_CH1)
- net OPTION: now also SW5.1
- net SCL: now reaches U2.42 (PB6/I2C1_SCL/TIM4_CH1/USART1_TX)
- net SCL: now also DS1.2 (SCL), R8.1
- net SDA: now reaches U2.43 (PB7/I2C1_SDA/TIM4_CH2/USART1_RX)
- net SDA: now also DS1.1 (SDA), R9.1
- new net: C21.1, DS1.3 (VCC), L3.1
- new net: L3.2, R7.1
- new net: C22.2, RV1.1
- new net: C23.2, RV1.4
- new net: J5.1, RV1.2
- new net: J5.2, RV1.5
- no-connect marks 14 -> 22
Other:
- note added: "OLED is super noisy. Needs its own GND return path and RCL filter."
- moved on the sheet: R2

Commit message: Footprints
Parts:
- C1, C2, C21: footprint (none) -> Capacitors_SMD:C_1206
- C10, C11, C12, C20, C3, C4, C5, C9: footprint (none) -> Capacitors_SMD:C_0805
- C13, C19, C22, C23, C6: footprint (none) -> Capacitors_SMD:CP_Elec_3x5.3
- C14, C15: value C_Small -> 100nF; footprint (none) -> Capacitors_SMD:C_0805
- C16, C17, C18, C7, C8: footprint (none) -> Capacitors_SMD:C_0603
- DS1: footprint (none) -> oled_display:128x32_OLED_I2C_Module
- J1: footprint (none) -> Connectors:USB_Mini-B
- J2: footprint (none) -> Pin_Headers:Pin_Header_Straight_2x03_Pitch2.54mm
- J3: footprint (none) -> customMicroSD:SOFNG_TF_15x15_PUSH_PUSH
- J4: footprint (none) -> Pin_Headers:Pin_Header_Straight_1x04_Pitch2.54mm
- J5: footprint (none) -> 35RAPC4BHN2:SWITCHCRAFT_35RAPC4BHN2
- L1: footprint (none) -> Inductors_SMD:L_0603
- L2, L3: footprint (none) -> custom_inductors:L_4x4
- R1, R2, R3, R4, R5, R6, R7, R8, R9: footprint (none) -> Resistors_SMD:R_0805
- RV1: footprint (none) -> Potentiometers:Potentiometer_Alps_RK097_Double_Vertical
- SW1, SW2, SW3, SW4, SW5: footprint (none) -> Buttons_Switches_THT:SW_TH_Tactile_Omron_B3F-10xx
- U3: footprint (none) -> Housings_SSOP:MSOP-10_3x3mm_Pitch0.5mm
- U4: footprint (none) -> Housings_SOIC:SOIC-24W_7.5x15.4mm_Pitch1.27mm
- U5: footprint (none) -> Housings_SOIC:SOIC-16W_5.3x10.2mm_Pitch1.27mm
- U6: footprint (none) -> Housings_SOIC:SOIC-14_3.9x8.7mm_Pitch1.27mm
- Y1: footprint (none) -> Crystals:Crystal_SMD_HC49-SD
Connections:
- net +3V3: now also U2.1 (VBAT)
- no-connect marks 22 -> 28

Commit message: PCB first pass
Parts:
- added H1, H2, H3, H4: M3, Mounting_Holes:MountingHole_3.2mm_M3, symbol mechanical:MountingHole
- J5: symbol conn:Audio-Jack-3 -> conn_custom:Audio-Jack-3
Connections:
- net +5V: now also U3.7 (VCC)
- net GND: now also J5.1; no longer J5.3
- net VCC: no longer U3.7 (VCC)
- net at RV1.2: now also J5.3; no longer J5.1
Changed lines of the file:
@@
 TX
-$Comp
-L power:VCC #PWR06
-U 1 1 5D059E10
-P 3150 8500
-F 0 "#PWR06" H 3150 8350 50  0001 C CNN
-F 1 "VCC" V 3167 8628 50  0000 L CNN
-F 2 "" H 3150 8500 50  0001 C CNN
-F 3 "" H 3150 8500 50  0001 C CNN
-	1    3150 8500
-	0    1    1    0
-$EndComp
 $Comp
 L power:GND #PWR02
@@
 $EndComp
 $Comp
-L conn:Audio-Jack-3 J5
+L conn_custom:Audio-Jack-3 J5
 U 1 1 5D14207F
 P 14550 7350
@@
 	0    -1   -1   0
 $EndComp
+$Comp
+L mechanical:MountingHole H1
+U 1 1 5D0CCC85
+P 4450 10150
+F 0 "H1" H 4550 10196 50  0000 L CNN
+F 1 "M3" H 4550 10105 50  0000 L CNN
+F 2 "Mounting_Holes:MountingHole_3.2mm_M3" H 4450 10150 50  0001 C CNN
+F 3 "~" H 4450 10150 50  0001 C CNN
+	1    4450 10150
+	1    0    0    -1
+$EndComp
+$Comp
+L mechanical:MountingHole H2
+U 1 1 5D0CCDCD
+P 4450 10350
+F 0 "H2" H 4550 10396 50  0000 L CNN
+F 1 "M3" H 4550 10305 50  0000 L CNN
+F 2 "Mounting_Holes:MountingHole_3.2mm_M3" H 4450 10350 50  0001 C CNN
+F 3 "~" H 4450 10350 50  0001 C CNN
+	1    4450 10350
+	1    0    0    -1
+$EndComp
+$Comp
+L mechanical:MountingHole H3
+U 1 1 5D0CCE57
+P 4450 10550
+F 0 "H3" H 4550 10596 50  0000 L CNN
+F 1 "M3" H 4550 10505 50  0000 L CNN
+F 2 "Mounting_Holes:MountingHole_3.2mm_M3" H 4450 10550 50  0001 C CNN
+F 3 "~" H 4450 10550 50  0001 C CNN
+	1    4450 10550
+	1    0    0    -1
+$EndComp
+$Comp
+L mechanical:MountingHole H4
+U 1 1 5D0CCEE7
+P 4450 10750
+F 0 "H4" H 4550 10796 50  0000 L CNN
+F 1 "M3" H 4550 10705 50  0000 L CNN
+F 2 "Mounting_Holes:MountingHole_3.2mm_M3" H 4450 10750 50  0001 C CNN
+F 3 "~" H 4450 10750 50  0001 C CNN
+	1    4450 10750
+	1    0    0    -1
+$EndComp
+$Comp
+L power:+5V #PWR0111
+U 1 1 5D0CF4B8
+P 3150 8500
+F 0 "#PWR0111" H 3150 8350 50  0001 C CNN
+F 1 "+5V" H 3165 8673 50  0000 C CNN
+F 2 "" H 3150 8500 50  0001 C CNN
+F 3 "" H 3150 8500 50  0001 C CNN
+	1    3150 8500
+	0    1    1    0
+$EndComp
 $EndSCHEMATC

Commit message: PCB first pass
Connections:
- net GND: now also U6.11 (V-); no longer U6.11 (V-)
Changed lines of the file:
@@
 L power:GNDA #PWR047
 U 1 1 5D08ABA3
-P 14750 5300
-F 0 "#PWR047" H 14750 5050 50  0001 C CNN
-F 1 "GNDA" H 14755 5127 50  0000 C CNN
-F 2 "" H 14750 5300 50  0001 C CNN
-F 3 "" H 14750 5300 50  0001 C CNN
-	1    14750 5300
+P 14750 2900
+F 0 "#PWR047" H 14750 2650 50  0001 C CNN
+F 1 "GNDA" H 14755 2727 50  0000 C CNN
+F 2 "" H 14750 2900 50  0001 C CNN
+F 3 "" H 14750 2900 50  0001 C CNN
+	1    14750 2900
 	1    0    0    -1
 $EndComp
@@
 	14550 2700 14550 2950
 Wire Wire Line
-	14550 2950 15150 2950
-Wire Wire Line
-	15150 2950 15150 2600
-Wire Wire Line
 	14550 2950 13900 2950
 Wire Wire Line
@@
 Wire Wire Line
 	13900 3500 13750 3500
-Connection ~ 14550 2950
 Wire Wire Line
 	13750 3600 13950 3600
@@
 	0    1    1    0
 $EndComp
+Wire Wire Line
+	15150 3050 14550 3050
+Wire Wire Line
+	14550 3050 14550 2950
+Wire Wire Line
+	15150 2600 15150 3050
+Connection ~ 14550 2950
 $EndSCHEMATC

Commit message: Added schematic images and pdf
Other:
- note added: "I/O"
- note added: "OPL3 and Analog Stage"
- note added: "UART and SD\n"
- note added: "USB & Power Filtering"
- moved on the sheet: C1, C12, C13, C2, C21, C3, C4, C5, C6, DS1, H1, H2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
